Commit message: update for wbr urdf

File: RobotURDFs/wbr_description/urdf/wbr_hand.urdf (robot description, URDF)
Before this commit: robot hand_robot, 11 links, 10 joints
Links:
- added link hand_base_link, mass 0.25; collision mesh filename=package://wbr_description/meshes/hand/R_hand.dae scale=0.001 0.001 0.001; visual mesh filename=package://wbr_description/meshes/hand/R_hand.STL scale=0.001 0.001 0.001
- link base_link: mass 0.25 -> 1.0; geometry collision box size=0.001 0.001 0.001; visual box size=0.001 0.001 0.001
- link index_finger_1: geometry collision mesh filename=package://wbr_description/meshes/hand/R_first_finger_F3.dae scale=0.001 0.001 0.001; visual mesh filename=package://wbr_description/meshes/hand/R_first_finger_F3.STL scale=0.001 0.001 0.001
- link index_finger_2: geometry collision mesh filename=package://wbr_description/meshes/hand/R_first_finger_F2.dae scale=0.001 0.001 0.001; visual mesh filename=package://wbr_description/meshes/hand/R_first_finger_F2.STL scale=0.001 0.001 0.001
- link index_finger_3: geometry collision mesh filename=package://wbr_description/meshes/hand/R_first_finger_F1.dae scale=0.001 0.001 0.001; visual mesh filename=package://wbr_description/meshes/hand/R_first_finger_F1.STL scale=0.001 0.001 0.001
- link middle_finger_1: geometry collision mesh filename=package://wbr_description/meshes/hand/R_middle_finger_F3.dae scale=0.001 0.001 0.001; visual mesh filename=package://wbr_description/meshes/hand/R_middle_finger_F3.STL scale=0.001 0.001 0.001
- link middle_finger_2: geometry collision mesh filename=package://wbr_description/meshes/hand/R_middle_finger_F2.dae scale=0.001 0.001 0.001; visual mesh filename=package://wbr_description/meshes/hand/R_middle_finger_F2.STL scale=0.001 0.001 0.001
- link middle_finger_3: geometry collision mesh filename=package://wbr_description/meshes/hand/R_middle_finger_F1.dae scale=0.001 0.001 0.001; visual mesh filename=package://wbr_description/meshes/hand/R_middle_finger_F1.STL scale=0.001 0.001 0.001
- link thumb_1: geometry collision mesh filename=package://wbr_description/meshes/hand/R_thumb_F4.dae scale=0.001 0.001 0.001; visual mesh filename=package://wbr_description/meshes/hand/R_thumb_F4.STL scale=0.001 0.001 0.001
- link thumb_2: geometry collision mesh filename=package://wbr_description/meshes/hand/R_thumb_F3.dae scale=0.001 0.001 0.001; visual mesh filename=package://wbr_description/meshes/hand/R_thumb_F3.STL scale=0.001 0.001 0.001
- link thumb_3: geometry collision mesh filename=package://wbr_description/meshes/hand/R_thumb_F2.dae scale=0.001 0.001 0.001; visual mesh filename=package://wbr_description/meshes/hand/R_thumb_F2.STL scale=0.001 0.001 0.001
- link thumb_4: geometry collision mesh filename=package://wbr_description/meshes/hand/R_thumb_F1.dae scale=0.001 0.001 0.001; visual mesh filename=package://wbr_description/meshes/hand/R_thumb_F1.STL scale=0.001 0.001 0.001
Joints:
- added joint hand_joint: type fixed, parent base_link, child hand_base_link, origin xyz=0 0.1 -0.07 rpy=0 0 1.57
- joint index_joint_1: parent base_link -> hand_base_link
- joint middle_joint_1: parent base_link -> hand_base_link
- joint thumb_joint_1: parent base_link -> hand_base_link
