Commit message: set grasp

File: RobotURDFs/finger_description/urdf/RH8D.urdf (robot description, URDF)
Before this commit: robot RH8D, 21 links, 20 joints
Links:
- link base_link: mass None -> 1.0; geometry collision box size=0.001 0.001 0.001; visual box size=0.001 0.001 0.001
Joints:
- joint palm__palm axis: origin xyz=-0.0265 0 -0.01025 rpy=0 0 0 -> xyz=-0.0265 0 -0.01025 rpy=0.6 0 0

File: RobotURDFs/wbr_description/urdf/wbr_hand_1.5.urdf (robot description, URDF)
Before this commit: robot hand_robot, 12 links, 11 joints
Links:
- link hand_base_link: geometry collision mesh filename=package://wbr_description/meshes/hand/R_hand.stl scale=0.001 0.001 0.001; visual mesh filename=package://wbr_description/meshes/hand/R_hand.STL scale=0.001 0.001 0.001
- link index_finger_1: geometry collision mesh filename=package://wbr_description/meshes/hand/R_first_finger_F3.stl scale=0.0015 0.001 0.001; visual mesh filename=package://wbr_description/meshes/hand/R_first_finger_F3.STL scale=0.0015 0.001 0.001
- link index_finger_2: geometry collision mesh filename=package://wbr_description/meshes/hand/R_first_finger_F2.stl scale=0.001 0.0015 0.001; visual mesh filename=package://wbr_description/meshes/hand/R_first_finger_F2.STL scale=0.001 0.0015 0.001
- link index_finger_3: geometry collision mesh filename=package://wbr_description/meshes/hand/R_first_finger_F1.stl scale=0.001 0.0015 0.001; visual mesh filename=package://wbr_description/meshes/hand/R_first_finger_F1.STL scale=0.001 0.0015 0.001
- link middle_finger_1: geometry collision mesh filename=package://wbr_description/meshes/hand/R_middle_finger_F3.stl scale=0.0015 0.001 0.001; visual mesh filename=package://wbr_description/meshes/hand/R_middle_finger_F3.STL scale=0.0015 0.001 0.001
- link middle_finger_2: geometry collision mesh filename=package://wbr_description/meshes/hand/R_middle_finger_F2.stl scale=0.001 0.0015 0.001; visual mesh filename=package://wbr_description/meshes/hand/R_middle_finger_F2.STL scale=0.001 0.0015 0.001
- link middle_finger_3: geometry collision mesh filename=package://wbr_description/meshes/hand/R_middle_finger_F1.stl scale=0.001 0.0015 0.001; visual mesh filename=package://wbr_description/meshes/hand/R_middle_finger_F1.STL scale=0.001 0.0015 0.001
- link thumb_3: geometry collision mesh filename=package://wbr_description/meshes/hand/R_thumb_F2.stl scale=0.001 0.0015 0.001; visual mesh filename=package://wbr_description/meshes/hand/R_thumb_F2.STL scale=0.001 0.0015 0.001
- link thumb_4: geometry collision mesh filename=package://wbr_description/meshes/hand/R_thumb_F1.stl scale=0.001 0.0015 0.001; visual mesh filename=package://wbr_description/meshes/hand/R_thumb_F1.STL scale=0.001 0.0015 0.001
Joints:
- joint hand_joint: origin xyz=0 -0.07 0.0 rpy=0 0 -1.57 -> xyz=0 -0.08 -0.01 rpy=0 0 -1.57
- joint index_joint_2: origin xyz=-0.02 0 0 rpy=0 1.57 -1.57 -> xyz=-0.03 0 0 rpy=0 1.57 -1.57
- joint index_joint_3: limit lower=0 upper=2.44 effort=1.0 velocity=1.0 -> lower=0 upper=1.57 effort=1.0 velocity=1.0; origin xyz=0.003 -0.0455 0 rpy=0 0 0 -> xyz=0.003 -0.06825 0 rpy=0 0 0
- joint middle_joint_2: limit lower=0 upper=1.75 effort=1.0 velocity=1.0 -> lower=0 upper=1.57 effort=1.0 velocity=1.0; origin xyz=-0.02 0 0 rpy=0 1.57 -1.57 -> xyz=-0.03 0 0 rpy=0 1.57 -1.57
- joint middle_joint_3: limit lower=0 upper=2.44 effort=1.0 velocity=1.0 -> lower=0 upper=1.57 effort=1.0 velocity=1.0; origin xyz=0.003 -0.0505 0 rpy=0 0 0 -> xyz=0.003 -0.06825 0 rpy=0 0 0
- joint thumb_joint_1: limit lower=0 upper=1.57 effort=1.0 velocity=1.0 -> lower=-1.57 upper=0 effort=1.0 velocity=1.0; origin xyz=0 0.0067 0.015 rpy=-1.57 -1.57 -1.57 -> xyz=0 0.0067 0.015 rpy=-1.57 0 -1.57
- joint thumb_joint_4: origin xyz=0.0045 -0.04 0 rpy=0 0 0 -> xyz=0.0045 -0.06 0 rpy=0 0 0

File: RobotURDFs/wbr_description/urdf/wbr_hand_2.0.urdf (robot description, URDF)
Before this commit: robot hand_robot, 12 links, 11 joints
Links:
- link hand_base_link: geometry collision mesh filename=package://wbr_description/meshes/hand/R_hand.stl scale=0.001 0.001 0.001; visual mesh filename=package://wbr_description/meshes/hand/R_hand.STL scale=0.001 0.001 0.001
- link index_finger_1: geometry collision mesh filename=package://wbr_description/meshes/hand/R_first_finger_F3.stl scale=0.002 0.001 0.001; visual mesh filename=package://wbr_description/meshes/hand/R_first_finger_F3.STL scale=0.002 0.001 0.001
- link index_finger_2: geometry collision mesh filename=package://wbr_description/meshes/hand/R_first_finger_F2.stl scale=0.001 0.002 0.001; visual mesh filename=package://wbr_description/meshes/hand/R_first_finger_F2.STL scale=0.001 0.002 0.001
- link index_finger_3: geometry collision mesh filename=package://wbr_description/meshes/hand/R_first_finger_F1.stl scale=0.001 0.002 0.001; visual mesh filename=package://wbr_description/meshes/hand/R_first_finger_F1.STL scale=0.001 0.002 0.001
- link middle_finger_1: geometry collision mesh filename=package://wbr_description/meshes/hand/R_middle_finger_F3.stl scale=0.002 0.001 0.001; visual mesh filename=package://wbr_description/meshes/hand/R_middle_finger_F3.STL scale=0.002 0.001 0.001
- link middle_finger_2: geometry collision mesh filename=package://wbr_description/meshes/hand/R_middle_finger_F2.stl scale=0.001 0.002 0.001; visual mesh filename=package://wbr_description/meshes/hand/R_middle_finger_F2.STL scale=0.001 0.002 0.001
- link middle_finger_3: geometry collision mesh filename=package://wbr_description/meshes/hand/R_middle_finger_F1.stl scale=0.001 0.002 0.001; visual mesh filename=package://wbr_description/meshes/hand/R_middle_finger_F1.STL scale=0.001 0.002 0.001
- link thumb_3: geometry collision mesh filename=package://wbr_description/meshes/hand/R_thumb_F2.stl scale=0.001 0.002 0.001; visual mesh filename=package://wbr_description/meshes/hand/R_thumb_F2.STL scale=0.001 0.002 0.001
- link thumb_4: geometry collision mesh filename=package://wbr_description/meshes/hand/R_thumb_F1.stl scale=0.001 0.002 0.001; visual mesh filename=package://wbr_description/meshes/hand/R_thumb_F1.STL scale=0.001 0.002 0.001
Joints:
- joint hand_joint: origin xyz=0 -0.07 0.0 rpy=0 0 -1.57 -> xyz=0 -0.1 -0.05 rpy=0 0 -1.57
- joint index_joint_2: origin xyz=-0.02 0 0 rpy=0 1.57 -1.57 -> xyz=-0.04 0 0 rpy=0 1.57 -1.57
- joint index_joint_3: limit lower=0 upper=2.44 effort=1.0 velocity=1.0 -> lower=0 upper=1.57 effort=1.0 velocity=1.0; origin xyz=0.003 -0.0455 0 rpy=0 0 0 -> xyz=0.003 -0.091 0 rpy=0 0 0
- joint middle_joint_2: limit lower=0 upper=1.75 effort=1.0 velocity=1.0 -> lower=0 upper=1.57 effort=1.0 velocity=1.0; origin xyz=-0.02 0 0 rpy=0 1.57 -1.57 -> xyz=-0.04 0 0 rpy=0 1.57 -1.57
- joint middle_joint_3: limit lower=0 upper=2.44 effort=1.0 velocity=1.0 -> lower=0 upper=1.57 effort=1.0 velocity=1.0; origin xyz=0.003 -0.0505 0 rpy=0 0 0 -> xyz=0.003 -0.091 0 rpy=0 0 0
- joint thumb_joint_1: limit lower=0 upper=1.57 effort=1.0 velocity=1.0 -> lower=-1.57 upper=0 effort=1.0 velocity=1.0; origin xyz=0 0.0067 0.015 rpy=-1.57 -1.57 -1.57 -> xyz=0 0.0067 0.015 rpy=-1.57 0 -1.57
- joint thumb_joint_4: origin xyz=0.0045 -0.04 0 rpy=0 0 0 -> xyz=0.0045 -0.08 0 rpy=0 0 0
