Commit message: change force control settings

File: ObjectURDFs/cylinder/cylinder.urdf (robot description, URDF)
Before this commit: robot cylinder.urdf, 1 links, 0 joints
Links:
- link cylinder: geometry collision cylinder length=0.03 radius=0.01; visual cylinder length=0.03 radius=0.01

File: RobotURDFs/wbr_description/urdf/wbr_hand.urdf (robot description, URDF)
Before this commit: robot hand_robot, 12 links, 11 joints
Links:
- link hand_base_link: geometry collision mesh filename=package://wbr_description/meshes/hand/R_hand.stl scale=0.001 0.001 0.001; visual mesh filename=package://wbr_description/meshes/hand/R_hand.STL scale=0.001 0.001 0.001
- link index_finger_1: geometry collision mesh filename=package://wbr_description/meshes/hand/R_first_finger_F3.stl scale=0.001 0.001 0.001; visual mesh filename=package://wbr_description/meshes/hand/R_first_finger_F3.STL scale=0.001 0.001 0.001
- link index_finger_2: geometry collision mesh filename=package://wbr_description/meshes/hand/R_first_finger_F2.stl scale=0.001 0.001 0.001; visual mesh filename=package://wbr_description/meshes/hand/R_first_finger_F2.STL scale=0.001 0.001 0.001
- link index_finger_3: geometry collision mesh filename=package://wbr_description/meshes/hand/R_first_finger_F1.stl scale=0.001 0.001 0.001; visual mesh filename=package://wbr_description/meshes/hand/R_first_finger_F1.STL scale=0.001 0.001 0.001
- link middle_finger_1: geometry collision mesh filename=package://wbr_description/meshes/hand/R_middle_finger_F3.stl scale=0.001 0.001 0.001; visual mesh filename=package://wbr_description/meshes/hand/R_middle_finger_F3.STL scale=0.001 0.001 0.001
- link middle_finger_2: geometry collision mesh filename=package://wbr_description/meshes/hand/R_middle_finger_F2.stl scale=0.001 0.001 0.001; visual mesh filename=package://wbr_description/meshes/hand/R_middle_finger_F2.STL scale=0.001 0.001 0.001
- link middle_finger_3: geometry collision mesh filename=package://wbr_description/meshes/hand/R_middle_finger_F1.stl scale=0.001 0.001 0.001; visual mesh filename=package://wbr_description/meshes/hand/R_middle_finger_F1.STL scale=0.001 0.001 0.001
- link thumb_1: geometry collision mesh filename=package://wbr_description/meshes/hand/R_thumb_F4.stl scale=0.001 0.001 0.001; visual mesh filename=package://wbr_description/meshes/hand/R_thumb_F4.STL scale=0.001 0.001 0.001
- link thumb_2: geometry collision mesh filename=package://wbr_description/meshes/hand/R_thumb_F3.stl scale=0.001 0.001 0.001; visual mesh filename=package://wbr_description/meshes/hand/R_thumb_F3.STL scale=0.001 0.001 0.001
- link thumb_3: geometry collision mesh filename=package://wbr_description/meshes/hand/R_thumb_F2.stl scale=0.001 0.001 0.001; visual mesh filename=package://wbr_description/meshes/hand/R_thumb_F2.STL scale=0.001 0.001 0.001
- link thumb_4: geometry collision mesh filename=package://wbr_description/meshes/hand/R_thumb_F1.stl scale=0.001 0.001 0.001; visual mesh filename=package://wbr_description/meshes/hand/R_thumb_F1.STL scale=0.001 0.001 0.001

Commit message: add cap with

File: ObjectURDFs/cylinder/cylinder.urdf (robot description, URDF)
Before this commit: robot cylinder.urdf, 1 links, 0 joints
Links:
- link cylinder: mass .1 -> 0.05; geometry collision mesh filename=package://cylinder/conicaltube050.stl scale=0.001 0.001 0.001; visual mesh filename=package://cylinder/conicaltube050.stl scale=0.001 0.001 0.001

File: ObjectURDFs/cylinder/cylinder_cap.urdf (robot description, URDF)
Before this commit: robot cylinder.urdf, 2 links, 1 joints
Joints:
- joint cap_joint: axis 0 0 1 -> 1 1 1

File: RobotURDFs/wbr_description/urdf/wbr_hand_with_cap.urdf (robot description, URDF)
Before this commit: robot hand_robot, 14 links, 13 joints
Links:
- link index_finger_3: geometry collision mesh filename=package://wbr_description/meshes/hand/R_first_finger_F1.stl scale=0.0007 0.0007 0.0007; visual mesh filename=package://wbr_description/meshes/hand/R_first_finger_F1.STL scale=0.001 0.001 0.001
- link thumb_4: geometry collision mesh filename=package://wbr_description/meshes/hand/R_thumb_F1.stl scale=0.0007 0.0007 0.0007; visual mesh filename=package://wbr_description/meshes/hand/R_thumb_F1.STL scale=0.001 0.001 0.001
Joints:
- joint thumb_joint_1: limit lower=0 upper=1.57 effort=1.0 velocity=1.0 -> lower=-1.57 upper=0 effort=1.0 velocity=1.0; origin xyz=0 0.0067 0.015 rpy=-1.57 -1.57 -1.57 -> xyz=0 0.0067 0.015 rpy=-1.57 0 -1.57
- joint thumb_joint_3: limit lower=0 upper=1.57 effort=1.0 velocity=1.0 -> lower=0 upper=3.14 effort=1.0 velocity=1.0
